File: KiCAD/SZG-TEMPLATE-TXR/SZG-TEMPLATE-TXR.sch (KiCad schematic (older format))
At the start: 28 parts, among them J1 SYZYGY_TXR-4, J2 Conn_01x06, U1 ATtiny44A-MU

Commit message: Corrected a net name. Improved example SYZYGY connector breakout routing for TXR board.
Connections:
- net labels added: RX3P
- net labels removed: RS3P
Changed lines of the file:
@@
 S8
 Text Label 1550 3850 0    50   ~ 0
-RS3P
+RX3P
 Text Label 1550 3950 0    50   ~ 0
 RX3N

Commit message: Updated the template projects MCU programming header to use the standard Tag-Connect cable pin order.
Connections:
- wire segments 72 -> 71
Changed lines of the file:
@@
 Wire Wire Line
 	6500 3500 7150 3500
-Text Label 9550 3300 0    50   ~ 0
+Text Label 9550 3400 0    50   ~ 0
 MCU_SCL_USCK
+Text Label 9550 3200 0    50   ~ 0
+MCU_MISO
 Text Label 9550 3500 0    50   ~ 0
-MCU_MISO
-Text Label 9550 3400 0    50   ~ 0
 MCU_SDA_MOSI
 Wire Wire Line
@@
 L power:+3.3V #PWR0110
 U 1 1 60652346
-P 9750 3150
-F 0 "#PWR0110" H 9750 3000 50  0001 C CNN
-F 1 "+3.3V" H 9765 3323 50  0000 C CNN
-F 2 "" H 9750 3150 50  0001 C CNN
-F 3 "" H 9750 3150 50  0001 C CNN
-	1    9750 3150
-	1    0    0    -1
+P 10150 3300
+F 0 "#PWR0110" H 10150 3150 50  0001 C CNN
+F 1 "+3.3V" H 10165 3473 50  0000 C CNN
+F 2 "" H 10150 3300 50  0001 C CNN
+F 3 "" H 10150 3300 50  0001 C CNN
+	1    10150 3300
+	0    1    1    0
 $EndComp
 $Comp
@@
 	-1   0    0    -1
 $EndComp
-Wire Wire Line
-	9500 3200 9750 3200
-Wire Wire Line
-	9750 3200 9750 3150
 Wire Wire Line
 	9500 3700 9750 3700
@@
 	1    0    0    -1
 $EndComp
+Wire Wire Line
+	9500 3200 10150 3200
 $EndSCHEMATC
